Commit message: modified camera tilt

File: replace_stuff_folder/hector_quadrotor_noetic/description/quadrotor_hokuyo_utm30lx.urdf.xacro (robot description, xacro)
@@ -14,5 +14,5 @@
     <xacro:include filename="$(find hector_sensors_description)/urdf/generic_camera.urdf.xacro" />
     <xacro:generic_camera name="front_cam" parent="base_link" ros_topic="camera/image" cam_info_topic="camera/camera_info" update_rate="3" res_x="512" res_y="512" image_format="R8G8B8" hfov="90">
-      <origin xyz="0.05 0.0 -0.06" rpy="0 0 0"/>
+      <origin xyz="0.05 0.0 -0.06" rpy="0 0.785 0"/>
     </xacro:generic_camera>
 </robot>

Commit message: camera pitch finalized at 0.7

File: replace_stuff_folder/hector_quadrotor_noetic/description/quadrotor_hokuyo_utm30lx.urdf.xacro (robot description, xacro)
@@ -14,5 +14,5 @@
     <xacro:include filename="$(find hector_sensors_description)/urdf/generic_camera.urdf.xacro" />
     <xacro:generic_camera name="front_cam" parent="base_link" ros_topic="camera/image" cam_info_topic="camera/camera_info" update_rate="3" res_x="512" res_y="512" image_format="R8G8B8" hfov="90">
-      <origin xyz="0.05 0.0 -0.06" rpy="0 0.785 0"/>
+      <origin xyz="0.05 0.0 -0.06" rpy="0 0.7 0"/>
     </xacro:generic_camera>
 </robot>
